File: Jupiter.kicad_sch (KiCad schematic)
At the start: 341 parts, among them J1 Conn_01x04, SW1 SW_Push, U1 ATmega32U4-M, Y1 Crystal_GND24_Small

Commit message: Placed keys on board
Connections:
- net COL0: now also U1.8 (PB0)
- net COL1: now also U1.9 (PB1)
- net COL10: now also U1.18 (PD0)
- net COL11: now also U1.19 (PD1)
- net COL12: now also U1.20 (PD2)
- net COL13: now also U1.21 (PD3)
- net COL14: now also U1.25 (PD4)
- net COL2: now also U1.10 (PB2)
- net COL3: now also U1.11 (PB3)
- net COL4: now also U1.28 (PB4)
- net COL5: now also U1.29 (PB5)
- net COL6: now also U1.30 (PB6)
- net COL7: now also U1.12 (PB7)
- net COL8: now also U1.31 (PC6)
- net COL9: now also U1.32 (PC7)
- net RGBLED: now also U1.37 (PF6)
- net ROW0: now also U1.22 (PD5)
- net ROW1: now also U1.26 (PD6)
- net ROW2: now also U1.41 (PF0)
- net ROW3: now also U1.40 (PF1)
- net ROW4: now also U1.39 (PF4)
- net ROW5: now also U1.38 (PF5)
Changed lines of the file:
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@@
+    )
+  )
+  (global_label "COL1" (shape input) (at 391.16 36.83 0) (fields_autoplaced)
+    (effects (font (size 1.27 1.27)) (justify left))
+    (property "Intersheet References" "${INTERSHEET_REFS}" (id 0) (at 398.4112 36.7506 0)
+      (effects (font (size 1.27 1.27)) (justify left) hide)
     )
   )
@@
     )
   )
+  (global_label "COL0" (shape input) (at 391.16 34.29 0) (fields_autoplaced)
+    (effects (font (size 1.27 1.27)) (justify left))
+    (property "Intersheet References" "${INTERSHEET_REFS}" (id 0) (at 398.4112 34.2106 0)
+      (effects (font (size 1.27 1.27)) (justify left) hide)
+    )
+  )
   (global_label "ROW3" (shape input) (at 29.21 95.25 180) (fields_autoplaced)
     (effects (font (size 1.27 1.27)) (justify right))
@@
     )
   )
+  (global_label "COL3" (shape input) (at 391.16 41.91 0) (fields_autoplaced)
+    (effects (font (size 1.27 1.27)) (justify left))
+    (property "Intersheet References" "${INTERSHEET_REFS}" (id 0) (at 398.4112 41.8306 0)
+      (effects (font (size 1.27 1.27)) (justify left) hide)
+    )
+  )
+  (global_label "ROW3" (shape input) (at 391.16 97.79 0) (fields_autoplaced)
+    (effects (font (size 1.27 1.27)) (justify left))
+    (property "Intersheet References" "${INTERSHEET_REFS}" (id 0) (at 398.8345 97.8694 0)
+      (effects (font (size 1.27 1.27)) (justify left) hide)
+    )
+  )
+  (global_label "ROW1" (shape input) (at 391.16 80.01 0) (fields_autoplaced)
+    (effects (font (size 1.27 1.27)) (justify left))
+    (property "Intersheet References" "${INTERSHEET_REFS}" (id 0) (at 398.8345 80.0894 0)
+      (effects (font (size 1.27 1.27)) (justify left) hide)
+    )
+  )
+  (global_label "COL13" (shape input) (at 391.16 72.39 0) (fields_autoplaced)
+    (effects (font (size 1.27 1.27)) (justify left))
+    (property "Intersheet References" "${INTERSHEET_REFS}" (id 0) (at 399.6207 72.3106 0)
+      (effects (font (size 1.27 1.27)) (justify left) hide)
+    )
+  )
   (global_label "COL9" (shape input) (at 195.58 21.59 90) (fields_autoplaced)
     (effects (font (size 1.27 1.27)) (justify left))
@@
     )
   )
+  (global_label "COL6" (shape input) (at 391.16 49.53 0) (fields_autoplaced)
+    (effects (font (size 1.27 1.27)) (justify left))
+    (property "Intersheet References" "${INTERSHEET_REFS}" (id 0) (at 398.4112 49.4506 0)
+      (effects (font (size 1.27 1.27)) (justify left) hide)
+    )
+  )
+  (global_label "COL11" (shape input) (at 391.16 67.31 0) (fields_autoplaced)
+    (effects (font (size 1.27 1.27)) (justify left))
+    (property "Intersheet References" "${INTERSHEET_REFS}" (id 0) (at 399.6207 67.2306 0)
+      (effects (font (size 1.27 1.27)) (justify left) hide)
+    )
+  )
+  (global_label "COL10" (shape input) (at 391.16 64.77 0) (fields_autoplaced)
+    (effects (font (size 1.27 1.27)) (justify left))
+    (property "Intersheet References" "${INTERSHEET_REFS}" (id 0) (at 399.6207 64.6906 0)
+      (effects (font (size 1.27 1.27)) (justify left) hide)
+    )
+  )
   (global_label "COL6" (shape input) (at 146.05 21.59 90) (fields_autoplaced)
     (effects (font (size 1.27 1.27)) (justify left))
@@
     )
   )
+  (global_label "COL2" (shape input) (at 391.16 39.37 0) (fields_autoplaced)
+    (effects (font (size 1.27 1.27)) (justify left))
+    (property "Intersheet References" "${INTERSHEET_REFS}" (id 0) (at 398.4112 39.2906 0)
+      (effects (font (size 1.27 1.27)) (justify left) hide)
+    )
+  )
+  (global_label "ROW5" (shape input) (at 391.16 102.87 0) (fields_autoplaced)
+    (effects (font (size 1.27 1.27)) (justify left))
+    (property "Intersheet References" "${INTERSHEET_REFS}" (id 0) (at 398.8345 102.9494 0)
+      (effects (font (size 1.27 1.27)) (justify left) hide)
+    )
+  )
   (global_label "COL5" (shape input) (at 128.27 21.59 90) (fields_autoplaced)
     (effects (font (size 1.27 1.27)) (justify left))
@@
     )
   )
+  (global_label "ROW0" (shape input) (at 391.16 77.47 0) (fields_autoplaced)
+    (effects (font (size 1.27 1.27)) (justify left))
+    (property "Intersheet References" "${INTERSHEET_REFS}" (id 0) (at 398.8345 77.5494 0)
+      (effects (font (size 1.27 1.27)) (justify left) hide)
+    )
+  )
   (global_label "D-" (shape input) (at 360.68 62.23 180) (fields_autoplaced)
     (effects (font (size 1.27 1.27)) (justify right))
@@
     )
   )
+  (global_label "ROW4" (shape input) (at 391.16 100.33 0) (fields_autoplaced)
+    (effects (font (size 1.27 1.27)) (justify left))
+    (property "Intersheet References" "${INTERSHEET_REFS}" (id 0) (at 398.8345 100.4094 0)
+      (effects (font (size 1.27 1.27)) (justify left) hide)
+    )
+  )
+  (global_label "RGBLED" (shape input) (at 391.16 105.41 0) (fields_autoplaced)
+    (effects (font (size 1.27 1.27)) (justify left))
+    (property "Intersheet References" "${INTERSHEET_REFS}" (id 0) (at 400.8302 105.4894 0)
+      (effects (font (size 1.27 1.27)) (justify left) hide)
+    )
+  )
+  (global_label "COL8" (shape input) (at 391.16 57.15 0) (fields_autoplaced)
+    (effects (font (size 1.27 1.27)) (justify left))
+    (property "Intersheet References" "${INTERSHEET_REFS}" (id 0) (at 398.4112 57.0706 0)
+      (effects (font (size 1.27 1.27)) (justify left) hide)
+    )
+  )
+  (global_label "COL4" (shape input) (at 391.16 44.45 0) (fields_autoplaced)
+    (effects (font (size 1.27 1.27)) (justify left))
+    (property "Intersheet References" "${INTERSHEET_REFS}" (id 0) (at 398.4112 44.3706 0)
+      (effects (font (size 1.27 1.27)) (justify left) hide)
+    )
+  )
   (global_label "COL7" (shape input) (at 162.56 21.59 90) (fields_autoplaced)
     (effects (font (size 1.27 1.27)) (justify left))
@@
     )
   )
+  (global_label "COL7" (shape input) (at 391.16 52.07 0) (fields_autoplaced)
+    (effects (font (size 1.27 1.27)) (justify left))
+    (property "Intersheet References" "${INTERSHEET_REFS}" (id 0) (at 398.4112 51.9906 0)
+      (effects (font (size 1.27 1.27)) (justify left) hide)
+    )
+  )
+  (global_label "COL9" (shape input) (at 391.16 59.69 0) (fields_autoplaced)
+    (effects (font (size 1.27 1.27)) (justify left))
+    (property "Intersheet References" "${INTERSHEET_REFS}" (id 0) (at 398.4112 59.6106 0)
+      (effects (font (size 1.27 1.27)) (justify left) hide)
+    )
+  )
   (global_label "ROW1" (shape input) (at 29.21 57.15 180) (fields_autoplaced)
     (effects (font (size 1.27 1.27)) (justify right))
@@
     )
   )
+  (global_label "ROW2" (shape input) (at 391.16 95.25 0) (fields_autoplaced)
+    (effects (font (size 1.27 1.27)) (justify left))
+    (property "Intersheet References" "${INTERSHEET_REFS}" (id 0) (at 398.8345 95.3294 0)
+      (effects (font (size 1.27 1.27)) (justify left) hide)
+    )
+  )
   (global_label "ROW5" (shape input) (at 29.21 133.35 180) (fields_autoplaced)
     (effects (font (size 1.27 1.27)) (justify right))
@@
     )
   )
+  (global_label "COL5" (shape input) (at 391.16 46.99 0) (fields_autoplaced)
+    (effects (font (size 1.27 1.27)) (justify left))
+    (property "Intersheet References" "${INTERSHEET_REFS}" (id 0) (at 398.4112 46.9106 0)
+      (effects (font (size 1.27 1.27)) (justify left) hide)
+    )
+  )
   (global_label "COL4" (shape input) (at 111.76 21.59 90) (fields_autoplaced)
     (effects (font (size 1.27 1.27)) (justify left))
@@
       (effects (font (size 1.27 1.27)) (justify left) hide)
     )
+  )
+  (global_label "COL12" (shape input) (at 391.16 69.85 0) (fields_autoplaced)
+    (effects (font (size 1.27 1.27)) (justify left))
+    (property "Intersheet References" "${INTERSHEET_REFS}" (id 0) (at 399.6207 69.7706 0)
+      (effects (font (size 1.27 1.27)) (justify left) hide)
+    )
+  )
+  (global_label "COL14" (shape input) (at 391.16 74.93 0) (fields_autoplaced)
+    (effects (font (size 1.27 1.27)) (justify left))
+    (property "Intersheet References" "${INTERSHEET_REFS}" (id 0) (at 399.6207 74.8506 0)
+      (effects (font (size 1.27 1.27)) (justify left) hide)
+    )

Commit message: Flipped LED footprint
Parts:
- LED_0, LED_1, LED_2, LED_3, LED_4, LED_5, LED_6, LED_7, LED_8, LED_9, LED_A1, LED_B1, LED_C1, LED_D1, LED_E1, LED_F1, LED_F10, LED_F11, LED_F12, LED_F13, LED_F2, LED_F3, LED_F4, LED_F5, LED_F6, LED_F7, LED_F8, LED_F9, LED_G1, LED_H1, LED_I1, LED_J1, LED_K1, LED_L1, LED_M1, LED_N1, LED_O1, LED_P1, LED_Q1, LED_R1, LED_S1, LED_T1, LED_U1, LED_V1, LED_W1, LED_X1, LED_Y1, LED_Z1, LED_backslash1, LED_backspace1, LED_capsLock1, LED_closeBracket1, LED_colon1, LED_comma1, LED_delete1, LED_downArrow1, LED_end1, LED_enter1, LED_equals1, LED_esc1, LED_function1, LED_home1, LED_leftAlt1, LED_leftArrow1, LED_leftControl1, LED_leftShift1, LED_minus1, LED_openBracket1, LED_period1, LED_pgDn1, LED_pgUp1, LED_questionMark1, LED_quote1, LED_rightAlt1, LED_rightArrow1, LED_rightControl1, LED_rightShift1, LED_space1, LED_tab1, LED_tilda1, LED_upArrow1, LED_windows1: footprint marbastlib-mx:LED_MX_6028R -> marbastlib-mx:LED_MX_6028R-FLIPPED

Commit message: Finished vertical matrix traces
Parts:
- LED_0, LED_1, LED_2, LED_3, LED_4, LED_5, LED_6, LED_7, LED_8, LED_9, LED_A1, LED_B1, LED_C1, LED_D1, LED_E1, LED_F1, LED_F10, LED_F11, LED_F12, LED_F13, LED_F2, LED_F3, LED_F4, LED_F5, LED_F6, LED_F7, LED_F8, LED_F9, LED_G1, LED_H1, LED_I1, LED_J1, LED_K1, LED_L1, LED_M1, LED_N1, LED_O1, LED_P1, LED_Q1, LED_R1, LED_S1, LED_T1, LED_U1, LED_V1, LED_W1, LED_X1, LED_Y1, LED_Z1, LED_backslash1, LED_backspace1, LED_capsLock1, LED_closeBracket1, LED_colon1, LED_comma1, LED_delete1, LED_downArrow1, LED_end1, LED_enter1, LED_equals1, LED_esc1, LED_function1, LED_home1, LED_leftAlt1, LED_leftArrow1, LED_leftControl1, LED_leftShift1, LED_minus1, LED_openBracket1, LED_period1, LED_pgDn1, LED_pgUp1, LED_questionMark1, LED_quote1, LED_rightAlt1, LED_rightArrow1, LED_rightControl1, LED_rightShift1, LED_space1, LED_tab1, LED_tilda1, LED_upArrow1, LED_windows1: footprint marbastlib-mx:LED_MX_6028R-FLIPPED -> marbastlib-mx:LED_MX_6028R
Connections:
- net +5V: now also LED_upArrow1.4 (VSS); no longer LED_upArrow1.1 (VDD)
- net GND: now also LED_upArrow1.1 (VDD); no longer LED_upArrow1.4 (VSS)
- net RGBLED: now also LED_delete1.3 (DIN); no longer LED_esc1.3 (DIN)
- net at LED_Q1.2 (DOUT): now also LED_tab1.3 (DIN); no longer LED_W1.3 (DIN)
- net at LED_Q1.3 (DIN): now also LED_W1.2 (DOUT); no longer LED_tab1.2 (DOUT)
- net at LED_F2.2 (DOUT): now also LED_F1.3 (DIN); no longer LED_F3.3 (DIN)
- net at LED_F2.3 (DIN): now also LED_F3.2 (DOUT); no longer LED_F1.2 (DOUT)
- net at LED_leftControl1.2 (DOUT): now also LED_windows1.3 (DIN)
- net at LED_leftControl1.3 (DIN): now also LED_leftShift1.2 (DOUT); no longer LED_windows1.2 (DOUT)
- net at LED_K1.2 (DOUT): now also LED_L1.3 (DIN); no longer LED_J1.3 (DIN)
- net at LED_K1.3 (DIN): now also LED_J1.2 (DOUT); no longer LED_L1.2 (DOUT)
- net at LED_leftArrow1.2 (DOUT): now also LED_downArrow1.3 (DIN); no longer LED_rightControl1.3 (DIN)
- net at LED_leftArrow1.3 (DIN): now also LED_rightControl1.2 (DOUT); no longer LED_downArrow1.2 (DOUT)
- net at LED_end1.2 (DOUT): now also LED_rightShift1.3 (DIN); no longer LED_rightArrow1.3 (DIN)
- net at LED_end1.3 (DIN): now also LED_pgDn1.2 (DOUT); no longer LED_upArrow1.2 (DOUT)
- net at LED_colon1.2 (DOUT): now also LED_quote1.3 (DIN); no longer LED_L1.3 (DIN)
- net at LED_F6.2 (DOUT): now also LED_F5.3 (DIN); no longer LED_F7.3 (DIN)
- net at LED_F6.3 (DIN): now also LED_F7.2 (DOUT); no longer LED_F5.2 (DOUT)
- net at LED_questionMark1.2 (DOUT): now also LED_period1.3 (DIN); no longer LED_rightShift1.3 (DIN)
- net at LED_questionMark1.3 (DIN): now also LED_rightShift1.2 (DOUT); no longer LED_period1.2 (DOUT)
- net at LED_4.2 (DOUT): now also LED_5.3 (DIN); no longer LED_3.3 (DIN)
- net at LED_4.3 (DIN): now also LED_3.2 (DOUT); no longer LED_5.2 (DOUT)
- net at LED_Z1.3 (DIN): now also LED_X1.2 (DOUT); no longer LED_leftShift1.2 (DOUT)
- net at LED_leftShift1.3 (DIN): now also LED_Z1.2 (DOUT); no longer LED_capsLock1.2 (DOUT)
- net at LED_minus1.2 (DOUT): now also LED_equals1.3 (DIN); no longer LED_0.3 (DIN)
- net at LED_minus1.3 (DIN): now also LED_0.2 (DOUT); no longer LED_equals1.2 (DOUT)
- net at LED_leftAlt1.2 (DOUT): now also LED_space1.3 (DIN); no longer LED_windows1.3 (DIN)
- net at LED_9.3 (DIN): now also LED_8.2 (DOUT); no longer LED_0.2 (DOUT)
- net at LED_9.2 (DOUT): now also LED_0.3 (DIN); no longer LED_8.3 (DIN)
- net at LED_upArrow1.3 (DIN): now also LED_pgDn1.3 (DIN); no longer LED_rightShift1.2 (DOUT)
- net at LED_S1.2 (DOUT): now also LED_D1.3 (DIN); no longer LED_A1.3 (DIN)
- net at LED_S1.3 (DIN): now also LED_A1.2 (DOUT); no longer LED_D1.2 (DOUT)
- net at LED_esc1.2 (DOUT): now also LED_tilda1.3 (DIN); no longer LED_F1.3 (DIN)
- net at LED_rightArrow1.2 (DOUT): no longer LED_downArrow1.3 (DIN)
- net at LED_F8.3 (DIN): now also LED_F9.2 (DOUT); no longer LED_F7.2 (DOUT)
- net at LED_home1.2 (DOUT): now also LED_pgUp1.3 (DIN); no longer LED_backspace1.3 (DIN)
- net at LED_home1.3 (DIN): now also LED_backspace1.2 (DOUT); no longer LED_delete1.2 (DOUT)
- net at LED_F4.3 (DIN): now also LED_F5.2 (DOUT); no longer LED_F3.2 (DOUT)
- net at LED_C1.2 (DOUT): now also LED_X1.3 (DIN); no longer LED_V1.3 (DIN)
- net at LED_C1.3 (DIN): now also LED_V1.2 (DOUT); no longer LED_X1.2 (DOUT)
- net at LED_F4.2 (DOUT): now also LED_F3.3 (DIN); no longer LED_F5.3 (DIN)
- net at LED_Y1.2 (DOUT): now also LED_T1.3 (DIN); no longer LED_U1.3 (DIN)
- net at LED_Y1.3 (DIN): now also LED_U1.2 (DOUT); no longer LED_T1.2 (DOUT)
- net at LED_function1.2 (DOUT): now also LED_rightControl1.3 (DIN); no longer LED_rightAlt1.3 (DIN)
- net at LED_function1.3 (DIN): now also LED_rightAlt1.2 (DOUT); no longer LED_rightControl1.2 (DOUT)
- net at LED_M1.2 (DOUT): now also LED_N1.3 (DIN); no longer LED_comma1.3 (DIN)
- net at LED_M1.3 (DIN): now also LED_comma1.2 (DOUT); no longer LED_N1.2 (DOUT)
- net at LED_F12.2 (DOUT): now also LED_F11.3 (DIN); no longer LED_delete1.3 (DIN)
- net at LED_R1.2 (DOUT): now also LED_E1.3 (DIN); no longer LED_T1.3 (DIN)
- net at LED_R1.3 (DIN): now also LED_T1.2 (DOUT); no longer LED_E1.2 (DOUT)
- net at LED_F8.2 (DOUT): now also LED_F7.3 (DIN); no longer LED_F9.3 (DIN)
- net at LED_2.2 (DOUT): now also LED_3.3 (DIN); no longer LED_1.3 (DIN)
- net at LED_2.3 (DIN): now also LED_1.2 (DOUT); no longer LED_3.2 (DOUT)
- net at LED_leftAlt1.3 (DIN): now also LED_windows1.2 (DOUT); no longer LED_space1.2 (DOUT)
- net at LED_F12.3 (DIN): now also LED_delete1.2 (DOUT); no longer LED_F11.2 (DOUT)
- net at LED_F10.2 (DOUT): now also LED_F9.3 (DIN); no longer LED_F11.3 (DIN)
- net at LED_enter1.3 (DIN): now also LED_quote1.2 (DOUT); no longer LED_pgDn1.2 (DOUT)
- net at LED_pgUp1.2 (DOUT): now also LED_backslash1.3 (DIN); no longer LED_pgDn1.3 (DIN)
- net at LED_colon1.3 (DIN): now also LED_L1.2 (DOUT); no longer LED_quote1.2 (DOUT)
- net at LED_enter1.2 (DOUT): now also LED_upArrow1.2 (DOUT); no longer LED_quote1.3 (DIN)
- net at LED_capsLock1.3 (DIN): now also LED_tab1.2 (DOUT); no longer LED_A1.2 (DOUT)
- net at LED_7.2 (DOUT): now also LED_8.3 (DIN); no longer LED_6.3 (DIN)
- net at LED_7.3 (DIN): now also LED_6.2 (DOUT); no longer LED_8.2 (DOUT)
- net at LED_F10.3 (DIN): now also LED_F11.2 (DOUT); no longer LED_F9.2 (DOUT)
- net at LED_tilda1.2 (DOUT): now also LED_1.3 (DIN); no longer LED_tab1.3 (DIN)
- net at LED_backslash1.2 (DOUT): now also LED_closeBracket1.3 (DIN); no longer LED_pgUp1.3 (DIN)
- net at LED_closeBracket1.2 (DOUT): now also LED_openBracket1.3 (DIN); no longer LED_backslash1.3 (DIN)
- net at LED_B1.3 (DIN): now also LED_N1.2 (DOUT); no longer LED_V1.2 (DOUT)
- net at LED_G1.2 (DOUT): now also LED_H1.3 (DIN); no longer LED_F13.3 (DIN)
- net at LED_G1.3 (DIN): now also LED_F13.2 (DOUT); no longer LED_H1.2 (DOUT)
- net at LED_openBracket1.2 (DOUT): now also LED_P1.3 (DIN); no longer LED_closeBracket1.3 (DIN)
- net at LED_B1.2 (DOUT): now also LED_V1.3 (DIN); no longer LED_N1.3 (DIN)
- net at LED_P1.2 (DOUT): now also LED_O1.3 (DIN); no longer LED_openBracket1.3 (DIN)
- net at LED_O1.2 (DOUT): now also LED_I1.3 (DIN); no longer LED_P1.3 (DIN)
- net at LED_I1.2 (DOUT): now also LED_U1.3 (DIN); no longer LED_O1.3 (DIN)
- new net: LED_F1.2 (DOUT), LED_esc1.3 (DIN)
- new net: LED_downArrow1.2 (DOUT), LED_rightArrow1.3 (DIN)
- new net: LED_backspace1.3 (DIN), LED_equals1.2 (DOUT)
- new net: LED_E1.2 (DOUT), LED_W1.3 (DIN)
- new net: LED_comma1.3 (DIN), LED_period1.2 (DOUT)
- new net: LED_A1.3 (DIN), LED_capsLock1.2 (DOUT)
- new net: LED_5.2 (DOUT), LED_6.3 (DIN)
- new net: LED_rightAlt1.3 (DIN), LED_space1.2 (DOUT)
- new net: LED_D1.2 (DOUT), LED_F13.3 (DIN)
- new net: LED_H1.2 (DOUT), LED_J1.3 (DIN)
Other:
- moved on the sheet: LED_0, LED_1, LED_2, LED_3, LED_4, LED_5, LED_6, LED_7, LED_8, LED_9, LED_A1, LED_B1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
