File: Jupiter.kicad_sch (KiCad schematic)
At the start: 347 parts, among them J1 Connector_USB_C_Receptacle_US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, SW1 SW_Push, U1 ATmega32U4-M, U2 PRTR5V0U2X, Y1 Crystal_GND24_Small

Commit message: Changed diode footprint
Parts:
- D1, D10, D11, D12, D13, D14, D15, D16, D17, D18, D19, D2, D20, D21, D22, D23, D24, D25, D26, D27, D28, D29, D3, D30, D31, D32, D33, D34, D35, D36, D37, D38, D39, D4, D40, D41, D42, D43, D44, D45, D46, D47, D48, D49, D5, D50, D51, D52, D53, D54, D55, D56, D57, D58, D59, D6, D60, D61, D62, D63, D64, D65, D66, D67, D68, D69, D7, D70, D71, D72, D73, D74, D75, D76, D77, D78, D79, D8, D80, D81, D82, D9: footprint Diode_SMD:D_0603_1608Metric -> Diode_SMD:D_SOD-123

Commit message: Added images
Parts:
- Y1: value Crystal_GND24_Small -> 16MHz
Connections:
- net GND: now also J1.A6 (D+), J1.B6 (D+), R4.1, U2.2 (IO1); no longer U2.1 (GND)
Other:
- moved on the sheet: C1, C10, C11, C12, C13, C14, C15, C16, C17, C18, C19, C2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
