File: Jupiter.kicad_pcb (KiCad board)
At the start: 2 copper layers, 314.3 x 123.8 mm, 341 parts, among them J1 Conn_01x04, SW1 SW_Push, U1 ATmega32U4-M, Y1 Crystal_GND24_Small

Commit message: Finished LED placement
Parts:
- moved LED_pgUp1 750.9 mm to (361.0, 125.1)
- moved LED_leftArrow1 708.3 mm to (318.1, 187.0)
- moved LED_pgDn1 701.3 mm to (361.0, 144.1)
- moved LED_rightShift1 674.1 mm to (306.2, 163.2)
- moved LED_closeBracket1 671.7 mm to (303.9, 125.1)
- moved LED_rightArrow1 670.3 mm to (356.2, 187.0)
- moved LED_F11 658.0 mm to (289.6, 82.3)
- moved LED_F10 647.8 mm to (270.6, 82.2)
- moved LED_backslash1 634.9 mm to (327.7, 125.1)
- moved LED_backspace1 634.6 mm to (322.9, 106.1)
- moved LED_colon1 632.5 mm to (270.6, 144.2)
- moved LED_home1 630.2 mm to (361.0, 106.1)
- moved LED_end1 626.5 mm to (361.0, 163.2)
- moved LED_rightControl1 623.8 mm to (294.3, 182.3)
- moved LED_F9 620.1 mm to (251.5, 82.3)
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
Commit message: Flipped LED footprint
Parts:
- C8, C9, D8, U1: moved to B.Cu
- moved U1 732.1 mm to (343.9, 142.3), turned to 180 degrees
- moved D8 604.7 mm to (217.1, 82.2), turned to 90 degrees
- moved C8 389.2 mm to (60.2, 82.2), turned to -90 degrees
- moved C9 364.8 mm to (83.7, 82.4), turned to -90 degrees
- moved C21 0.19 mm to (-232.1, 218.3)
Routing:
- net GND: track 0.00 -> 15.3 mm

Commit message: Finished diode placement
Parts:
- D1, D10, D11, D12, D13, D14, D15, D16, D17, D18, D19, D2, D20, D21, D22, D23, D24, D25, D26, D27, D28, D29, D3, D30, D31, D32, D33, D34, D35, D36, D37, D38, D39, D4, D40, D41, D42, D43, D44, D45, D46, D47, D48, D49, D5, D50, D51, D52, D53, D54, D55, D56, D57, D58, D59, D6, D60, D61, D62, D63, D64, D65, D66, D67, D68, D69, D7, D70, D71, D72, D73, D74, D75, D76, D77, D78, D79, D80, D81, D82, D9: moved to B.Cu
- LED_0, LED_1, LED_2, LED_3, LED_4, LED_5, LED_6, LED_7, LED_8, LED_9, LED_A1, LED_B1, LED_C1, LED_D1, LED_E1, LED_F1, LED_F10, LED_F11, LED_F12, LED_F13, LED_F2, LED_F3, LED_F4, LED_F5, LED_F6, LED_F7, LED_F8, LED_F9, LED_G1, LED_H1, LED_I1, LED_J1, LED_K1, LED_L1, LED_M1, LED_N1, LED_O1, LED_P1, LED_Q1, LED_R1, LED_S1, LED_T1, LED_U1, LED_V1, LED_W1, LED_X1, LED_Y1, LED_Z1, LED_backslash1, LED_backspace1, LED_capsLock1, LED_closeBracket1, LED_colon1, LED_comma1, LED_delete1, LED_downArrow1, LED_end1, LED_enter1, LED_equals1, LED_esc1, LED_function1, LED_home1, LED_leftAlt1, LED_leftArrow1, LED_leftControl1, LED_leftShift1, LED_minus1, LED_openBracket1, LED_period1, LED_pgDn1, LED_pgUp1, LED_questionMark1, LED_quote1, LED_rightAlt1, LED_rightArrow1, LED_rightControl1, LED_rightShift1, LED_space1, LED_tab1, LED_tilda1, LED_upArrow1, LED_windows1: footprint marbastlib-mx:LED_MX_6028R -> marbastlib-mx:LED_MX_6028R-FLIPPED
- moved D72 744.2 mm to (368.0, 158.9), turned to 90 degrees
- moved D71 735.3 mm to (344.2, 163.7), turned to 90 degrees
- moved D82 705.5 mm to (363.2, 182.7), turned to 90 degrees
- moved D44 705.0 mm to (368.0, 120.8), turned to 90 degrees
- moved D81 694.0 mm to (344.2, 182.7), turned to 90 degrees
- moved D13 691.1 mm to (315.6, 78.0), turned to 90 degrees
- moved D14 688.8 mm to (339.4, 78.0), turned to 90 degrees
- moved D43 683.3 mm to (334.7, 120.8), turned to 90 degrees
- moved D42 683.0 mm to (310.9, 120.8), turned to 90 degrees
- moved D58 681.2 mm to (368.0, 139.9), turned to 90 degrees
- moved D29 678.8 mm to (368.0, 101.8), turned to 90 degrees
- moved D78 668.4 mm to (282.3, 178.0), turned to 90 degrees
- moved D26 663.2 mm to (282.3, 101.8), turned to 90 degrees
- moved D80 659.0 mm to (325.1, 182.8), turned to 90 degrees
- moved D28 653.3 mm to (329.9, 101.9), turned to 90 degrees
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Routing:
- net ROW4: track 0.00 -> 295.2 mm
- net ROW5: track 0.00 -> 276.2 mm
- net ROW0: track 0.00 -> 275.1 mm
- net ROW2: track 0.00 -> 265.7 mm
- net ROW1: track 0.00 -> 265.6 mm
- net ROW3: track 0.00 -> 255.8 mm
- net +5V: track 0.00 -> 33.9 mm
- net Net-(LED_esc1-Pad2): track 0.00 -> 19.0 mm
- net GND: track 15.3 -> 27.7 mm
- net Net-(K_esc1-Pad2): track 0.00 -> 5.67 mm
- net Net-(K_backspace1-Pad2): track 0.00 -> 5.57 mm
- net Net-(K_leftArrow1-Pad2): track 0.00 -> 5.56 mm
- net Net-(K_B1-Pad2): track 0.00 -> 5.56 mm
- net Net-(K_S1-Pad2): track 0.00 -> 5.56 mm
- net Net-(K_W1-Pad2): track 0.00 -> 5.50 mm
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
Commit message: Finished vertical matrix traces
Parts:
- C10, C11, C12, C13, C14, C15, C16, C17, C18, C19, C20, C21, C22: moved to B.Cu
- LED_0, LED_1, LED_2, LED_3, LED_4, LED_5, LED_6, LED_7, LED_8, LED_9, LED_A1, LED_B1, LED_C1, LED_D1, LED_E1, LED_F1, LED_F10, LED_F11, LED_F12, LED_F13, LED_F2, LED_F3, LED_F4, LED_F5, LED_F6, LED_F7, LED_F8, LED_F9, LED_G1, LED_H1, LED_I1, LED_J1, LED_K1, LED_L1, LED_M1, LED_N1, LED_O1, LED_P1, LED_Q1, LED_R1, LED_S1, LED_T1, LED_U1, LED_V1, LED_W1, LED_X1, LED_Y1, LED_Z1, LED_backslash1, LED_backspace1, LED_capsLock1, LED_closeBracket1, LED_colon1, LED_comma1, LED_delete1, LED_downArrow1, LED_end1, LED_enter1, LED_equals1, LED_esc1, LED_function1, LED_home1, LED_leftAlt1, LED_leftArrow1, LED_leftControl1, LED_leftShift1, LED_minus1, LED_openBracket1, LED_period1, LED_pgDn1, LED_pgUp1, LED_questionMark1, LED_quote1, LED_rightAlt1, LED_rightArrow1, LED_rightControl1, LED_rightShift1, LED_space1, LED_tab1, LED_tilda1, LED_upArrow1, LED_windows1: footprint marbastlib-mx:LED_MX_6028R-FLIPPED -> marbastlib-mx:LED_MX_6028R
- moved C20 610.8 mm to (314.5, 82.3), turned to -90 degrees
- moved C19 589.6 mm to (295.5, 82.3), turned to -90 degrees
- moved C21 586.4 mm to (338.3, 82.3), turned to -90 degrees
- moved C18 577.8 mm to (276.5, 82.1), turned to -90 degrees
- moved C16 524.5 mm to (233.5, 82.2), turned to -90 degrees
- moved C17 524.5 mm to (257.5, 82.1), turned to -90 degrees
- moved C14 511.8 mm to (195.5, 82.2), turned to -90 degrees
- moved C15 479.3 mm to (214.5, 82.2), turned to -90 degrees
- moved C13 452.2 mm to (176.5, 82.2), turned to -90 degrees
- moved C10 426.2 mm to (114.6, 82.2), turned to -90 degrees
- moved C11 416.6 mm to (133.8, 82.1), turned to -90 degrees
- moved C22 361.4 mm to (71.7, 106.1), turned to 90 degrees
- moved C12 186.0 mm to (152.6, 82.1), turned to -90 degrees
- moved C9 11.8 mm to (95.5, 82.2), turned to -90 degrees
- moved C8 11.7 mm to (71.7, 82.0), turned to -90 degrees
Connections:
- LED_0 pad 2: Net-(LED_9-Pad3) -> Net-(LED_0-Pad2)
- LED_1 pad 2: Net-(LED_tilda1-Pad3) -> Net-(LED_1-Pad2)
- LED_2 pad 2: Net-(LED_1-Pad3) -> Net-(LED_2-Pad2)
- LED_2 pad 3: Net-(LED_2-Pad3) -> Net-(LED_1-Pad2)
- LED_3 pad 2: Net-(LED_2-Pad3) -> Net-(LED_3-Pad2)
- LED_3 pad 3: Net-(LED_3-Pad3) -> Net-(LED_2-Pad2)
- LED_4 pad 2: Net-(LED_3-Pad3) -> Net-(LED_4-Pad2)
- LED_4 pad 3: Net-(LED_4-Pad3) -> Net-(LED_3-Pad2)
- LED_5 pad 2: Net-(LED_4-Pad3) -> Net-(LED_5-Pad2)
- LED_5 pad 3: Net-(LED_5-Pad3) -> Net-(LED_4-Pad2)
- LED_6 pad 2: Net-(LED_5-Pad3) -> Net-(LED_6-Pad2)
- LED_6 pad 3: Net-(LED_6-Pad3) -> Net-(LED_5-Pad2)
- LED_7 pad 2: Net-(LED_6-Pad3) -> Net-(LED_7-Pad2)
- LED_7 pad 3: Net-(LED_7-Pad3) -> Net-(LED_6-Pad2)
- LED_8 pad 2: Net-(LED_7-Pad3) -> Net-(LED_8-Pad2)
- LED_8 pad 3: Net-(LED_8-Pad3) -> Net-(LED_7-Pad2)
- LED_9 pad 2: Net-(LED_8-Pad3) -> Net-(LED_0-Pad3)
- LED_9 pad 3: Net-(LED_9-Pad3) -> Net-(LED_8-Pad2)
- LED_A1 pad 2: Net-(LED_capsLock1-Pad3) -> Net-(LED_A1-Pad2)
- LED_B1 pad 3: Net-(LED_V1-Pad2) -> Net-(LED_B1-Pad3)
- LED_C1 pad 3: Net-(LED_X1-Pad2) -> Net-(LED_C1-Pad3)
- LED_D1 pad 2: Net-(LED_S1-Pad3) -> Net-(LED_D1-Pad2)
- LED_E1 pad 3: Net-(LED_W1-Pad2) -> Net-(LED_E1-Pad3)
- LED_F1 pad 3: Net-(LED_esc1-Pad2) -> Net-(LED_F1-Pad3)
- LED_F10 pad 3: Net-(LED_F9-Pad2) -> Net-(LED_F10-Pad3)
- LED_F11 pad 2: Net-(LED_F11-Pad2) -> Net-(LED_F10-Pad3)
- LED_F11 pad 3: Net-(LED_F10-Pad2) -> Net-(LED_F11-Pad3)
- LED_F12 pad 2: Net-(LED_F12-Pad2) -> Net-(LED_F11-Pad3)
- LED_F12 pad 3: Net-(LED_F11-Pad2) -> Net-(LED_F12-Pad3)
- LED_F13 pad 2: Net-(LED_D1-Pad3) -> Net-(LED_F13-Pad2)
- LED_F13 pad 3: Net-(LED_F13-Pad3) -> Net-(LED_D1-Pad2)
- LED_F2 pad 2: Net-(LED_F2-Pad2) -> Net-(LED_F1-Pad3)
- LED_F2 pad 3: Net-(LED_F1-Pad2) -> Net-(LED_F2-Pad3)
- LED_F3 pad 2: Net-(LED_F3-Pad2) -> Net-(LED_F2-Pad3)
- LED_F3 pad 3: Net-(LED_F2-Pad2) -> Net-(LED_F3-Pad3)
- LED_F4 pad 2: Net-(LED_F4-Pad2) -> Net-(LED_F3-Pad3)
- LED_F4 pad 3: Net-(LED_F3-Pad2) -> Net-(LED_F4-Pad3)
- LED_F5 pad 2: Net-(LED_F5-Pad2) -> Net-(LED_F4-Pad3)
- LED_F5 pad 3: Net-(LED_F4-Pad2) -> Net-(LED_F5-Pad3)
- LED_F6 pad 2: Net-(LED_F6-Pad2) -> Net-(LED_F5-Pad3)
- LED_F6 pad 3: Net-(LED_F5-Pad2) -> Net-(LED_F6-Pad3)
- LED_F7 pad 2: Net-(LED_F7-Pad2) -> Net-(LED_F6-Pad3)
- LED_F7 pad 3: Net-(LED_F6-Pad2) -> Net-(LED_F7-Pad3)
- LED_F8 pad 2: Net-(LED_F8-Pad2) -> Net-(LED_F7-Pad3)
- LED_F8 pad 3: Net-(LED_F7-Pad2) -> Net-(LED_F8-Pad3)
- LED_F9 pad 2: Net-(LED_F9-Pad2) -> Net-(LED_F8-Pad3)
- LED_F9 pad 3: Net-(LED_F8-Pad2) -> Net-(LED_F10-Pad2)
- LED_G1 pad 2: Net-(LED_F13-Pad3) -> Net-(LED_G1-Pad2)
- LED_G1 pad 3: Net-(LED_G1-Pad3) -> Net-(LED_F13-Pad2)
- LED_H1 pad 2: Net-(LED_G1-Pad3) -> Net-(LED_H1-Pad2)
- LED_H1 pad 3: Net-(LED_H1-Pad3) -> Net-(LED_G1-Pad2)
- LED_I1 pad 3: Net-(LED_U1-Pad2) -> Net-(LED_I1-Pad3)
- LED_J1 pad 2: Net-(LED_H1-Pad3) -> Net-(LED_J1-Pad2)
- LED_J1 pad 3: Net-(LED_J1-Pad3) -> Net-(LED_H1-Pad2)
- LED_K1 pad 2: Net-(LED_J1-Pad3) -> Net-(LED_K1-Pad2)
- LED_K1 pad 3: Net-(LED_K1-Pad3) -> Net-(LED_J1-Pad2)
- LED_L1 pad 2: Net-(LED_K1-Pad3) -> Net-(LED_L1-Pad2)
- LED_L1 pad 3: Net-(LED_L1-Pad3) -> Net-(LED_K1-Pad2)
- LED_M1 pad 3: Net-(LED_N1-Pad2) -> Net-(LED_M1-Pad3)
- LED_N1 pad 2: Net-(LED_N1-Pad2) -> Net-(LED_B1-Pad3)
- LED_N1 pad 3: Net-(LED_B1-Pad2) -> Net-(LED_M1-Pad2)
- LED_O1 pad 2: Net-(LED_O1-Pad2) -> Net-(LED_I1-Pad3)
- LED_O1 pad 3: Net-(LED_I1-Pad2) -> Net-(LED_O1-Pad3)
- LED_P1 pad 2: Net-(LED_P1-Pad2) -> Net-(LED_O1-Pad3)
- LED_P1 pad 3: Net-(LED_O1-Pad2) -> Net-(LED_P1-Pad3)
- LED_Q1 pad 3: Net-(LED_tab1-Pad2) -> Net-(LED_Q1-Pad3)
- LED_R1 pad 2: Net-(LED_R1-Pad2) -> Net-(LED_E1-Pad3)
- LED_R1 pad 3: Net-(LED_E1-Pad2) -> Net-(LED_R1-Pad3)
- LED_S1 pad 2: Net-(LED_A1-Pad3) -> Net-(LED_D1-Pad3)
- LED_S1 pad 3: Net-(LED_S1-Pad3) -> Net-(LED_A1-Pad2)
- LED_T1 pad 2: Net-(LED_T1-Pad2) -> Net-(LED_R1-Pad3)
- LED_T1 pad 3: Net-(LED_R1-Pad2) -> Net-(LED_T1-Pad3)
- LED_U1 pad 3: Net-(LED_Y1-Pad2) -> Net-(LED_I1-Pad2)
- LED_V1 pad 2: Net-(LED_V1-Pad2) -> Net-(LED_C1-Pad3)
- LED_V1 pad 3: Net-(LED_C1-Pad2) -> Net-(LED_B1-Pad2)
- LED_W1 pad 2: Net-(LED_W1-Pad2) -> Net-(LED_Q1-Pad3)
- LED_W1 pad 3: Net-(LED_Q1-Pad2) -> Net-(LED_E1-Pad2)
- LED_X1 pad 3: Net-(LED_Z1-Pad2) -> Net-(LED_C1-Pad2)
- LED_Y1 pad 2: Net-(LED_Y1-Pad2) -> Net-(LED_T1-Pad3)
- LED_Y1 pad 3: Net-(LED_T1-Pad2) -> Net-(LED_U1-Pad2)
- LED_Z1 pad 3: Net-(LED_leftShift1-Pad2) -> Net-(LED_X1-Pad2)
- LED_backslash1 pad 3: Net-(LED_closeBracket1-Pad2) -> Net-(LED_backslash1-Pad3)
- LED_backspace1 pad 2: Net-(LED_equals1-Pad3) -> Net-(LED_backspace1-Pad2)
- LED_capsLock1 pad 2: Net-(LED_capsLock1-Pad2) -> Net-(LED_A1-Pad3)
- LED_closeBracket1 pad 3: Net-(LED_openBracket1-Pad2) -> Net-(LED_backslash1-Pad2)
- LED_colon1 pad 2: Net-(LED_L1-Pad3) -> Net-(LED_colon1-Pad2)
- LED_colon1 pad 3: Net-(LED_colon1-Pad3) -> Net-(LED_L1-Pad2)
- LED_comma1 pad 2: Net-(LED_comma1-Pad2) -> Net-(LED_M1-Pad3)
- LED_comma1 pad 3: Net-(LED_M1-Pad2) -> Net-(LED_comma1-Pad3)
- LED_delete1 pad 2: Net-(LED_delete1-Pad2) -> Net-(LED_F12-Pad3)
- LED_delete1 pad 3: Net-(LED_F12-Pad2) -> RGBLED
- LED_downArrow1 pad 2: Net-(LED_leftArrow1-Pad3) -> Net-(LED_downArrow1-Pad2)
- LED_end1 pad 2: Net-(LED_end1-Pad2) -> Net-(LED_rightShift1-Pad3)
- LED_end1 pad 3: Net-(LED_upArrow1-Pad2) -> Net-(LED_pgDn1-Pad2)
- LED_enter1 pad 2: Net-(LED_quote1-Pad3) -> Net-(LED_enter1-Pad2)
- LED_equals1 pad 2: Net-(LED_minus1-Pad3) -> Net-(LED_backspace1-Pad3)
- LED_esc1 pad 3: RGBLED -> Net-(LED_F1-Pad2)
- LED_function1 pad 2: Net-(LED_rightAlt1-Pad3) -> Net-(LED_function1-Pad2)
- LED_home1 pad 2: Net-(LED_backspace1-Pad3) -> Net-(LED_home1-Pad2)
- LED_home1 pad 3: Net-(LED_delete1-Pad2) -> Net-(LED_backspace1-Pad2)
- LED_leftAlt1 pad 2: Net-(LED_windows1-Pad3) -> Net-(LED_leftAlt1-Pad2)
- LED_leftArrow1 pad 2: Net-(LED_rightControl1-Pad3) -> Net-(LED_downArrow1-Pad3)
- LED_leftControl1 pad 2: unconnected-(LED_leftControl1-Pad2) -> Net-(LED_leftControl1-Pad2)
- LED_leftControl1 pad 3: Net-(LED_leftControl1-Pad3) -> Net-(LED_leftShift1-Pad2)
- LED_leftShift1 pad 3: Net-(LED_capsLock1-Pad2) -> Net-(LED_Z1-Pad2)
- LED_minus1 pad 2: Net-(LED_0-Pad3) -> Net-(LED_equals1-Pad3)
- LED_minus1 pad 3: Net-(LED_minus1-Pad3) -> Net-(LED_0-Pad2)
- LED_openBracket1 pad 2: Net-(LED_openBracket1-Pad2) -> Net-(LED_P1-Pad3)
- LED_openBracket1 pad 3: Net-(LED_P1-Pad2) -> Net-(LED_closeBracket1-Pad2)
- LED_period1 pad 2: Net-(LED_period1-Pad2) -> Net-(LED_comma1-Pad3)
- LED_period1 pad 3: Net-(LED_comma1-Pad2) -> Net-(LED_period1-Pad3)
- LED_pgDn1 pad 2: Net-(LED_enter1-Pad3) -> Net-(LED_pgDn1-Pad2)
- LED_pgDn1 pad 3: Net-(LED_pgUp1-Pad2) -> Net-(LED_pgDn1-Pad3)
- LED_pgUp1 pad 2: Net-(LED_pgUp1-Pad2) -> Net-(LED_backslash1-Pad3)
- LED_pgUp1 pad 3: Net-(LED_backslash1-Pad2) -> Net-(LED_home1-Pad2)
- LED_questionMark1 pad 2: Net-(LED_questionMark1-Pad2) -> Net-(LED_period1-Pad3)
- LED_questionMark1 pad 3: Net-(LED_period1-Pad2) -> Net-(LED_questionMark1-Pad3)
- LED_quote1 pad 2: Net-(LED_colon1-Pad3) -> Net-(LED_enter1-Pad3)
- LED_quote1 pad 3: Net-(LED_quote1-Pad3) -> Net-(LED_colon1-Pad2)
- LED_rightAlt1 pad 2: Net-(LED_space1-Pad3) -> Net-(LED_function1-Pad3)
- LED_rightArrow1 pad 2: Net-(LED_downArrow1-Pad3) -> unconnected-(LED_rightArrow1-Pad2)
- LED_rightArrow1 pad 3: Net-(LED_end1-Pad2) -> Net-(LED_downArrow1-Pad2)
- LED_rightControl1 pad 2: Net-(LED_function1-Pad3) -> Net-(LED_leftArrow1-Pad3)
- LED_rightControl1 pad 3: Net-(LED_rightControl1-Pad3) -> Net-(LED_function1-Pad2)
- LED_rightShift1 pad 2: Net-(LED_rightShift1-Pad2) -> Net-(LED_questionMark1-Pad3)
- LED_rightShift1 pad 3: Net-(LED_questionMark1-Pad2) -> Net-(LED_rightShift1-Pad3)
- LED_space1 pad 2: Net-(LED_leftAlt1-Pad3) -> Net-(LED_rightAlt1-Pad3)
- LED_space1 pad 3: Net-(LED_space1-Pad3) -> Net-(LED_leftAlt1-Pad2)
- LED_tab1 pad 2: Net-(LED_tab1-Pad2) -> Net-(LED_capsLock1-Pad3)
- LED_tab1 pad 3: Net-(LED_tilda1-Pad2) -> Net-(LED_Q1-Pad2)
- LED_tilda1 pad 2: Net-(LED_tilda1-Pad2) -> Net-(LED_1-Pad3)
- LED_tilda1 pad 3: Net-(LED_tilda1-Pad3) -> Net-(LED_esc1-Pad2)
- LED_upArrow1 pad 1: +5V -> GND
- LED_upArrow1 pad 2: Net-(LED_upArrow1-Pad2) -> Net-(LED_enter1-Pad2)
- LED_upArrow1 pad 3: Net-(LED_rightShift1-Pad2) -> Net-(LED_pgDn1-Pad3)
- LED_upArrow1 pad 4: GND -> +5V
- LED_windows1 pad 2: Net-(LED_leftControl1-Pad3) -> Net-(LED_leftAlt1-Pad3)
- LED_windows1 pad 3: Net-(LED_windows1-Pad3) -> Net-(LED_leftControl1-Pad2)
Routing:
- net GND: track 27.7 -> 282.5 mm
- net +5V: track 33.9 -> 288.3 mm
- net COL12: track 0.00 -> 128.7 mm
- net COL11: track 0.00 -> 128.2 mm
- net COL9: track 0.00 -> 124.7 mm
- net COL8: track 0.00 -> 122.8 mm
- net COL1: track 0.00 -> 121.5 mm
- net COL2: track 0.00 -> 119.4 mm
- net COL5: track 0.00 -> 114.8 mm
- net COL13: track 0.00 -> 114.6 mm
- net COL0: track 0.00 -> 110.3 mm
- net COL10: track 0.00 -> 98.2 mm
- net COL7: track 0.00 -> 96.1 mm
- net COL6: track 0.00 -> 94.7 mm
- net COL3: track 0.00 -> 94.1 mm
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
Commit message: Finished LED capacitor placement
Parts:
- C23, C24, C25, C26, C27, C28, C29, C30, C31, C32, C33, C34, C35, C36, C37, C38, C39, C40, C41, C42, C43, C44, C45, C46, C47, C48, C49, C50, C51, C52, C53, C54, C55, C56, C57, C58, C59, C60, C61, C62, C63, C64, C65, C66, C67, C68, C69, C70, C71, C72, C73, C74, C75, C76, C77, C78, C79, C80, C81, C82, C83, C84, C85, C86, C87, C88, C89, Y1: moved to B.Cu
- LED_0, LED_1, LED_2, LED_3, LED_4, LED_5, LED_6, LED_7, LED_8, LED_9, LED_A1, LED_D1, LED_F13, LED_G1, LED_H1, LED_J1, LED_K1, LED_L1, LED_S1, LED_backspace1, LED_capsLock1, LED_colon1, LED_downArrow1, LED_end1, LED_enter1, LED_equals1, LED_function1, LED_leftAlt1, LED_leftArrow1, LED_leftControl1, LED_minus1, LED_pgDn1, LED_pgUp1, LED_quote1, LED_rightAlt1, LED_rightArrow1, LED_rightControl1, LED_space1, LED_tilda1, LED_windows1: footprint marbastlib-mx:LED_MX_6028R -> marbastlib-mx:LED_MX_6028R-FLIPPED
- moved Y1 713.8 mm to (333.5, 147.5), turned to -45 degrees
- moved C89 690.1 mm to (367.0, 106.0), turned to -90 degrees
- moved C87 649.3 mm to (355.4, 144.2), turned to 90 degrees
- moved C35 636.8 mm to (317.0, 106.1), turned to 90 degrees
- moved C88 630.5 mm to (355.2, 125.1), turned to 90 degrees
- moved C83 630.0 mm to (312.2, 187.0), turned to 90 degrees
- moved C37 627.1 mm to (309.9, 125.0), turned to -90 degrees
- moved C34 625.2 mm to (288.4, 106.1), turned to 90 degrees
- moved C74 619.6 mm to (312.2, 163.1), turned to -90 degrees
- moved C86 614.6 mm to (355.6, 163.2), turned to 90 degrees
- moved C85 600.0 mm to (350.3, 187.0), turned to 90 degrees
- moved C84 593.1 mm to (331.4, 187.0), turned to 90 degrees
- moved C75 589.6 mm to (343.2, 167.9), turned to -90 degrees
- moved C40 578.6 mm to (252.7, 125.0), turned to -90 degrees
- moved C82 574.3 mm to (288.5, 182.3), turned to 90 degrees
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Connections:
- C2 pad 1: GND -> Net-(C2-Pad1)
- LED_backspace1 pad 2: Net-(LED_backspace1-Pad2) -> Net-(LED_backslash1-Pad3)
- LED_delete1 pad 3: RGBLED -> Net-(LED_delete1-Pad3)
- LED_end1 pad 2: Net-(LED_rightShift1-Pad3) -> Net-(LED_end1-Pad2)
- LED_end1 pad 3: Net-(LED_pgDn1-Pad2) -> RGBLED
- LED_home1 pad 2: Net-(LED_home1-Pad2) -> Net-(LED_delete1-Pad3)
- LED_home1 pad 3: Net-(LED_backspace1-Pad2) -> Net-(LED_home1-Pad3)
- LED_pgDn1 pad 3: Net-(LED_pgDn1-Pad3) -> Net-(LED_end1-Pad2)
- LED_pgUp1 pad 2: Net-(LED_backslash1-Pad3) -> Net-(LED_home1-Pad3)
- LED_pgUp1 pad 3: Net-(LED_home1-Pad2) -> Net-(LED_pgDn1-Pad2)
- LED_upArrow1 pad 1: GND -> +5V
- LED_upArrow1 pad 2: Net-(LED_enter1-Pad2) -> Net-(LED_rightShift1-Pad3)
- LED_upArrow1 pad 3: Net-(LED_pgDn1-Pad3) -> Net-(LED_enter1-Pad2)
- LED_upArrow1 pad 4: +5V -> GND
- U1 pad 16: GND -> Net-(C2-Pad1)
- Y1 pad 3: GND -> Net-(C2-Pad1)
Routing:
- net +5V: track 288.3 -> 1956.8 mm
- net GND: track 282.5 -> 1917.4 mm
- net Net-(LED_leftAlt1-Pad2): track 0.00 -> 66.6 mm
- net Net-(LED_rightAlt1-Pad3): track 0.00 -> 64.2 mm
- net Net-(LED_enter1-Pad2): track 0.00 -> 43.7 mm
- net Net-(LED_end1-Pad2): track 0.00 -> 40.9 mm
- net Net-(LED_pgDn1-Pad2): track 0.00 -> 40.3 mm
- net Net-(LED_delete1-Pad3): track 0.00 -> 38.6 mm
- net COL13: track 114.6 -> 85.8 mm
- net Net-(LED_rightShift1-Pad3): track 0.00 -> 28.2 mm
- net Net-(LED_home1-Pad3): track 0.00 -> 27.5 mm
- net Net-(LED_enter1-Pad3): track 0.00 -> 26.2 mm
- net Net-(LED_Z1-Pad2): track 0.00 -> 26.1 mm
- net Net-(LED_capsLock1-Pad3): track 0.00 -> 25.3 mm
- net ROW4: track 295.2 -> 270.5 mm, vias 0 -> 1
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
Commit message: added stabilizers
Parts:
- added REF**: STAB_MX_2.25u, marbastlib-mx:STAB_MX_2.25u, F.Cu at (320.6, 139.1)
- added REF**: STAB_MX_2u, marbastlib-mx:STAB_MX_2u, F.Cu at (322.9, 101.0)
- added REF**: STAB_MX_2.25u, marbastlib-mx:STAB_MX_2.25u, F.Cu at (77.7, 158.2)
- added REF**: STAB_MX_P_6.25u, marbastlib-mx:STAB_MX_P_6.25u, F.Cu at (187.2, 177.2)
- J1: moved to B.Cu
- moved J1 746.4 mm to (339.1, 90.2), turned to 90 degrees
- moved Y1 7.21 mm to (338.6, 142.4)
- moved U1 5.60 mm to (343.5, 137.7)
Routing:
- net COL0: track 110.3 -> 392.0 mm
- net ROW1: track 265.6 -> 545.7 mm
- net COL1: track 121.5 -> 397.3 mm
- net COL2: track 119.4 -> 364.1 mm
- net COL3: track 94.1 -> 321.9 mm
- net COL4: track 92.9 -> 297.8 mm
- net COL5: track 114.8 -> 299.9 mm
- net Net-(LED_backslash1-Pad3): track 22.7 -> 31.2 mm
- net COL11: track 128.2 -> 135.9 mm
- net COL12: track 128.7 -> 135.8 mm
- net GND: track 1917.4 -> 1918.7 mm
- net +5V: track 1956.8 -> 1957.4 mm
