File: Jupiter.kicad_pcb (KiCad board)
At the start: 2 copper layers, 314.3 x 123.8 mm, 345 parts, among them J1 Conn_01x04, SW1 SW_Push, U1 ATmega32U4-M, Y1 Crystal_GND24_Small

Commit message: Added traces
Parts:
- C1, C2, C3, C6, R1, R2, SW1: moved to B.Cu
- moved SW1 745.0 mm to (349.2, 160.2), turned to -90 degrees
- moved C3 666.4 mm to (348.2, 141.8), turned to -45 degrees
- moved R1 644.8 mm to (343.6, 147.3), turned to 45 degrees
- moved C2 639.1 mm to (341.6, 145.3), turned to 45 degrees
- moved R2 636.1 mm to (341.1, 131.8), turned to 135 degrees
- moved C6 627.1 mm to (337.1, 134.5), turned to -45 degrees
- moved C1 577.3 mm to (335.6, 139.5), turned to -135 degrees
- moved J1 9.24 mm to (346.8, 85.1)
Routing:
- net COL6: track 94.7 -> 279.5 mm
- net COL7: track 96.1 -> 261.2 mm
- net COL8: track 122.8 -> 267.9 mm
- net COL9: track 124.7 -> 249.8 mm
- net COL10: track 98.2 -> 203.3 mm
- net COL11: track 135.9 -> 212.2 mm
- net COL12: track 135.8 -> 192.9 mm
- net +5V: track 1957.4 -> 2006.1 mm, vias 0 -> 6
- net COL13: track 85.8 -> 117.8 mm
- net COL0: track 392.0 -> 415.7 mm
- net GND: track 1918.7 -> 1941.8 mm
- net COL2: track 364.1 -> 384.0 mm
- net COL5: track 299.9 -> 319.7 mm
- net COL4: track 297.8 -> 317.6 mm
- net Net-(R1-Pad2): track 0.00 -> 18.2 mm
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
Commit message: traces
Parts:
- removed REF** (x2): STAB_MX_2.25u, marbastlib-mx:STAB_MX_2.25u
- removed REF**: STAB_MX_2u, marbastlib-mx:STAB_MX_2u
- removed REF**: STAB_MX_P_6.25u, marbastlib-mx:STAB_MX_P_6.25u
- C4, C5, C7: moved to B.Cu
- moved C4 637.0 mm to (349.7, 134.1), turned to -135 degrees
- moved C7 622.5 mm to (343.1, 129.9), turned to 135 degrees
- moved C5 592.1 mm to (342.5, 146.0), turned to -135 degrees
- moved C1 4.19 mm to (332.4, 142.2)
- moved Y1 4.18 mm to (335.4, 145.1)
- moved C2 4.08 mm to (338.5, 148.1)
- moved J1 1.55 mm to (345.2, 84.7)
- moved C3 1.01 mm to (348.6, 142.8)
- moved R2 0.85 mm to (341.7, 131.2)
Connections:
- U1 pad 10: COL2 -> ROW4
- U1 pad 11: COL3 -> ROW5
- U1 pad 12: COL7 -> RGBLED
- U1 pad 19: COL11 -> COL7
- U1 pad 22: ROW0 -> COL11
- U1 pad 26: ROW1 -> unconnected-(U1-Pad26)
- U1 pad 36: unconnected-(U1-Pad36) -> COL3
- U1 pad 37: RGBLED -> COL2
- U1 pad 38: ROW5 -> COL1
- U1 pad 39: ROW4 -> ROW1
- U1 pad 40: ROW3 -> COL0
- U1 pad 41: ROW2 -> ROW0
- U1 pad 8: COL0 -> ROW3
- U1 pad 9: COL1 -> ROW2
Routing:
- net ROW0: track 275.1 -> 601.0 mm, vias 0 -> 2
- net +5V: track 2006.1 -> 2100.8 mm, vias 6 -> 8
- net GND: track 1941.8 -> 2036.1 mm
- net ROW4: track 270.5 -> 322.9 mm, vias 1 -> 2
- net ROW5: track 295.9 -> 341.7 mm, vias 0 -> 2
- net Net-(LED_leftControl1-Pad3): track 0.00 -> 34.9 mm
- net COL0: track 415.7 -> 447.6 mm
- net ROW1: track 558.9 -> 590.3 mm
- net Net-(LED_delete1-Pad3): track 22.1 -> 53.5 mm
- net RGBLED: track 4.76 -> 36.2 mm
- net COL1: track 406.0 -> 437.0 mm
- net COL2: track 384.0 -> 414.6 mm
- net COL3: track 338.7 -> 368.8 mm
- net ROW2: track 265.7 -> 276.3 mm, vias 0 -> 2
- net Net-(C2-Pad1): track 8.48 -> 12.9 mm
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
Commit message: more traces
Parts:
- added REF**: STAB_MX_2.25u, marbastlib-mx:STAB_MX_2.25u, F.Cu at (77.7, 158.2)
- added REF**: STAB_MX_P_6.25u, marbastlib-mx:STAB_MX_P_6.25u, F.Cu at (187.2, 177.2)
- added REF**: STAB_MX_2.25u, marbastlib-mx:STAB_MX_2.25u, F.Cu at (320.6, 139.1)
- added REF**: STAB_MX_2u, marbastlib-mx:STAB_MX_2u, F.Cu at (322.9, 101.0)
- moved Y1 1.50 mm to (336.3, 143.9)
- moved C2 1.45 mm to (339.4, 146.8)
- moved C1 1.44 mm to (333.1, 140.8)
- moved C6 0.29 mm to (336.8, 134.6), turned to 135 degrees
Connections:
- U1 pad 18: COL10 -> unconnected-(U1-Pad18)
- U1 pad 19: COL7 -> unconnected-(U1-Pad19)
- U1 pad 20: COL12 -> ROW2
- U1 pad 22: COL11 -> COL12
- U1 pad 25: COL14 -> COL11
- U1 pad 26: unconnected-(U1-Pad26) -> COL10
- U1 pad 27: unconnected-(U1-Pad27) -> COL9
- U1 pad 28: COL4 -> COL8
- U1 pad 29: COL5 -> COL7
- U1 pad 31: COL8 -> COL5
- U1 pad 32: COL9 -> COL4
- U1 pad 8: ROW3 -> COL14
- U1 pad 9: ROW2 -> ROW3
Routing:
- net ROW2: track 276.3 -> 324.5 mm, vias 2 -> 3
- net ROW1: track 590.3 -> 629.7 mm, vias 0 -> 2
- net COL13: track 117.8 -> 155.2 mm
- net COL12: track 192.9 -> 228.9 mm
- net COL11: track 212.2 -> 246.6 mm
- net COL10: track 203.3 -> 236.2 mm
- net COL9: track 249.8 -> 282.2 mm
- net COL8: track 267.9 -> 299.9 mm
- net COL7: track 261.2 -> 292.8 mm
- net COL6: track 279.5 -> 310.9 mm
- net COL5: track 319.7 -> 350.7 mm
- net COL4: track 317.6 -> 348.3 mm
- net COL14: track 82.9 -> 87.0 mm
- net GND: track 2036.1 -> 2040.0 mm
- net COL0: track 447.6 -> 450.7 mm
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
Commit message: almost finished trace routing
Connections:
- U1 pad 19: unconnected-(U1-Pad19) -> ROW3
- U1 pad 8: COL14 -> unconnected-(U1-Pad8)
- U1 pad 9: ROW3 -> COL14
Routing:
- net ROW3: track 259.6 -> 326.1 mm, vias 0 -> 2
- net COL13: track 155.2 -> 184.6 mm
- net COL14: track 87.0 -> 101.6 mm
- net GND: track 2040.0 -> 2046.7 mm
- net unconnected-(U1-Pad8): track 0.00 -> 4.04 mm
- net +5V: track 2102.2 -> 2102.4 mm, vias 8 -> 9

Commit message: edge cuts
Routing:
- net GND: track 2046.7 -> 2126.1 mm
- net D+: track 3.98 -> 68.5 mm
- net D-: track 3.68 -> 68.2 mm
- net Net-(LED_esc1-Pad2): track 0.00 -> 30.0 mm
- net +5V: track 2102.4 -> 2131.0 mm
- net unconnected-(U1-Pad8): track 4.04 -> 0.00 mm
- net COL0: track 450.7 -> 449.2 mm, vias 0 -> 1
Other:
- board size 314.3 x 123.8 mm -> 314.4 x 123.9 mm
