File: Jupiter.kicad_pcb (KiCad board)
At the start: 2 copper layers, 314.4 x 123.9 mm, 345 parts, among them J1 Conn_01x04, SW1 SW_Push, U1 ATmega32U4-M, Y1 Crystal_GND24_Small

Commit message: Finished usb-c assembly
Parts:
- added F1: 500mA, Fuse:Fuse_1206_3216Metric, B.Cu at (350.5, 82.9)
- added R3: 22, Resistor_SMD:R_0603_1608Metric, B.Cu at (353.8, 82.4)
- added R4: 22, Resistor_SMD:R_0603_1608Metric, B.Cu at (355.8, 82.4)
- added R5: 5.1k, Resistor_SMD:R_0603_1608Metric, B.Cu at (350.6, 78.7)
- added R6: 5.1k, Resistor_SMD:R_0603_1608Metric, B.Cu at (358.9, 78.8)
- added U2: PRTR5V0U2X, random-keyboard-parts:SOT143B, B.Cu at (354.8, 79.1)
- J1: value Conn_01x04 -> Connector_USB_C_Receptacle_USB2.0; footprint random-keyboard-parts:JST-SR-4 -> marbastlib-various:USB_C_Receptacle_HRO_TYPE-C-31-M-14
- moved J1 14.3 mm to (354.7, 74.0), turned to 0 degrees
Routing:
- net +5V: track 2131.0 -> 2102.3 mm, vias 9 -> 7
- net Net-(LED_delete1-Pad3): track 53.5 -> 34.3 mm
- net VBUS: track 0.00 -> 15.3 mm, vias 0 -> 2
- net GND: track 2126.1 -> 2140.0 mm
- net Net-(J1-PadA6): track 0.00 -> 9.61 mm
- net Net-(J1-PadA7): track 0.00 -> 8.27 mm
- net Net-(J1-PadA5): track 0.00 -> 5.71 mm, vias 0 -> 2
- net Net-(J1-PadB5): track 0.00 -> 5.45 mm, vias 0 -> 2
- net D-: track 68.2 -> 63.6 mm
- net D+: track 68.5 -> 64.2 mm
Other:
- outline, holes or cut-outs redrawn

Commit message: Corrected LED orientation
Parts:
- LED_0, LED_1, LED_2, LED_3, LED_4, LED_5, LED_6, LED_7, LED_8, LED_9, LED_A1, LED_D1, LED_F13, LED_G1, LED_H1, LED_J1, LED_K1, LED_L1, LED_S1, LED_backspace1, LED_capsLock1, LED_colon1, LED_downArrow1, LED_end1, LED_enter1, LED_equals1, LED_function1, LED_leftAlt1, LED_leftArrow1, LED_leftControl1, LED_minus1, LED_pgDn1, LED_pgUp1, LED_quote1, LED_rightAlt1, LED_rightArrow1, LED_rightControl1, LED_space1, LED_tilda1, LED_windows1: footprint marbastlib-mx:LED_MX_6028R-FLIPPED -> marbastlib-mx:LED_MX_6028R
- LED_B1, LED_C1, LED_E1, LED_F1, LED_F10, LED_F11, LED_F12, LED_F2, LED_F3, LED_F4, LED_F5, LED_F6, LED_F7, LED_F8, LED_F9, LED_I1, LED_M1, LED_N1, LED_O1, LED_P1, LED_Q1, LED_R1, LED_T1, LED_U1, LED_V1, LED_W1, LED_X1, LED_Y1, LED_Z1, LED_backslash1, LED_closeBracket1, LED_comma1, LED_delete1, LED_esc1, LED_home1, LED_leftShift1, LED_openBracket1, LED_period1, LED_questionMark1, LED_rightShift1, LED_tab1, LED_upArrow1: footprint marbastlib-mx:LED_MX_6028R -> marbastlib-mx:LED_MX_6028R-FLIPPED
- moved C21 29.1 mm to (355.1, 106.1), turned to 90 degrees
- moved C86 24.7 mm to (362.2, 187.0), turned to -90 degrees
- moved C88 22.4 mm to (367.0, 144.1), turned to -90 degrees
- moved C87 22.3 mm to (367.0, 163.2), turned to -90 degrees
- moved C89 19.0 mm to (367.0, 125.1)
- turned C10 to 90 degrees
- turned C11 to 90 degrees
- turned C12 to 90 degrees
- turned C13 to 90 degrees
- turned C14 to 90 degrees
- turned C15 to 90 degrees
- turned C16 to 90 degrees
- turned C17 to 90 degrees
- turned C18 to 90 degrees
- turned C19 to 90 degrees
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Connections:
- J1 pad A6: Net-(J1-PadA6) -> GND
- J1 pad B6: Net-(J1-PadA6) -> GND
- LED_2 pad 2: Net-(LED_2-Pad2) -> Net-(LED_1-Pad3)
- LED_2 pad 3: Net-(LED_1-Pad2) -> Net-(LED_2-Pad3)
- LED_3 pad 2: Net-(LED_3-Pad2) -> Net-(LED_2-Pad3)
- LED_3 pad 3: Net-(LED_2-Pad2) -> Net-(LED_3-Pad3)
- LED_4 pad 2: Net-(LED_4-Pad2) -> Net-(LED_3-Pad3)
- LED_4 pad 3: Net-(LED_3-Pad2) -> Net-(LED_4-Pad3)
- LED_5 pad 2: Net-(LED_5-Pad2) -> Net-(LED_4-Pad3)
- LED_5 pad 3: Net-(LED_4-Pad2) -> Net-(LED_5-Pad3)
- LED_6 pad 2: Net-(LED_6-Pad2) -> Net-(LED_5-Pad3)
- LED_6 pad 3: Net-(LED_5-Pad2) -> Net-(LED_6-Pad3)
- LED_7 pad 2: Net-(LED_7-Pad2) -> Net-(LED_6-Pad3)
- LED_7 pad 3: Net-(LED_6-Pad2) -> Net-(LED_7-Pad3)
- LED_8 pad 2: Net-(LED_8-Pad2) -> Net-(LED_7-Pad3)
- LED_8 pad 3: Net-(LED_7-Pad2) -> Net-(LED_8-Pad3)
- LED_9 pad 2: Net-(LED_0-Pad3) -> Net-(LED_8-Pad3)
- LED_9 pad 3: Net-(LED_8-Pad2) -> Net-(LED_0-Pad2)
- LED_F11 pad 2: Net-(LED_F10-Pad3) -> Net-(LED_F11-Pad2)
- LED_F11 pad 3: Net-(LED_F11-Pad3) -> Net-(LED_F10-Pad2)
- LED_F12 pad 2: Net-(LED_F11-Pad3) -> Net-(LED_F12-Pad2)
- LED_F12 pad 3: Net-(LED_F12-Pad3) -> Net-(LED_F11-Pad2)
- LED_F13 pad 2: Net-(LED_F13-Pad2) -> Net-(LED_D1-Pad3)
- LED_F13 pad 3: Net-(LED_D1-Pad2) -> Net-(LED_F13-Pad3)
- LED_F2 pad 2: Net-(LED_F1-Pad3) -> Net-(LED_F2-Pad2)
- LED_F2 pad 3: Net-(LED_F2-Pad3) -> Net-(LED_F1-Pad2)
- LED_F3 pad 2: Net-(LED_F2-Pad3) -> Net-(LED_F3-Pad2)
- LED_F3 pad 3: Net-(LED_F3-Pad3) -> Net-(LED_F2-Pad2)
- LED_F4 pad 2: Net-(LED_F3-Pad3) -> Net-(LED_F4-Pad2)
- LED_F4 pad 3: Net-(LED_F4-Pad3) -> Net-(LED_F3-Pad2)
- LED_F5 pad 2: Net-(LED_F4-Pad3) -> Net-(LED_F5-Pad2)
- LED_F5 pad 3: Net-(LED_F5-Pad3) -> Net-(LED_F4-Pad2)
- LED_F6 pad 2: Net-(LED_F5-Pad3) -> Net-(LED_F6-Pad2)
- LED_F6 pad 3: Net-(LED_F6-Pad3) -> Net-(LED_F5-Pad2)
- LED_F7 pad 2: Net-(LED_F6-Pad3) -> Net-(LED_F7-Pad2)
- LED_F7 pad 3: Net-(LED_F7-Pad3) -> Net-(LED_F6-Pad2)
- LED_F8 pad 2: Net-(LED_F7-Pad3) -> Net-(LED_F8-Pad2)
- LED_F8 pad 3: Net-(LED_F8-Pad3) -> Net-(LED_F7-Pad2)
- LED_F9 pad 2: Net-(LED_F8-Pad3) -> Net-(LED_F10-Pad3)
- LED_F9 pad 3: Net-(LED_F10-Pad2) -> Net-(LED_F8-Pad2)
- LED_G1 pad 2: Net-(LED_G1-Pad2) -> Net-(LED_F13-Pad3)
- LED_G1 pad 3: Net-(LED_F13-Pad2) -> Net-(LED_G1-Pad3)
- LED_H1 pad 2: Net-(LED_H1-Pad2) -> Net-(LED_G1-Pad3)
- LED_H1 pad 3: Net-(LED_G1-Pad2) -> Net-(LED_H1-Pad3)
- LED_J1 pad 2: Net-(LED_J1-Pad2) -> Net-(LED_H1-Pad3)
- LED_J1 pad 3: Net-(LED_H1-Pad2) -> Net-(LED_J1-Pad3)
- LED_K1 pad 2: Net-(LED_K1-Pad2) -> Net-(LED_J1-Pad3)
- LED_K1 pad 3: Net-(LED_J1-Pad2) -> Net-(LED_K1-Pad3)
- LED_L1 pad 2: Net-(LED_L1-Pad2) -> Net-(LED_K1-Pad3)
- LED_L1 pad 3: Net-(LED_K1-Pad2) -> Net-(LED_L1-Pad3)
- LED_N1 pad 2: Net-(LED_B1-Pad3) -> Net-(LED_M1-Pad3)
- LED_N1 pad 3: Net-(LED_M1-Pad2) -> Net-(LED_B1-Pad2)
- LED_O1 pad 2: Net-(LED_I1-Pad3) -> Net-(LED_O1-Pad2)
- LED_O1 pad 3: Net-(LED_O1-Pad3) -> Net-(LED_I1-Pad2)
- LED_P1 pad 2: Net-(LED_O1-Pad3) -> Net-(LED_P1-Pad2)
- LED_P1 pad 3: Net-(LED_P1-Pad3) -> Net-(LED_O1-Pad2)
- LED_R1 pad 2: Net-(LED_E1-Pad3) -> Net-(LED_R1-Pad2)
- LED_R1 pad 3: Net-(LED_R1-Pad3) -> Net-(LED_E1-Pad2)
- LED_S1 pad 2: Net-(LED_D1-Pad3) -> Net-(LED_A1-Pad3)
- LED_S1 pad 3: Net-(LED_A1-Pad2) -> Net-(LED_D1-Pad2)
- LED_T1 pad 2: Net-(LED_R1-Pad3) -> Net-(LED_T1-Pad2)
- LED_T1 pad 3: Net-(LED_T1-Pad3) -> Net-(LED_R1-Pad2)
- LED_U1 pad 2: Net-(LED_U1-Pad2) -> Net-(LED_I1-Pad3)
- LED_U1 pad 3: Net-(LED_I1-Pad2) -> Net-(LED_U1-Pad3)
- LED_V1 pad 2: Net-(LED_C1-Pad3) -> Net-(LED_B1-Pad3)
- LED_V1 pad 3: Net-(LED_B1-Pad2) -> Net-(LED_C1-Pad2)
- LED_W1 pad 2: Net-(LED_Q1-Pad3) -> Net-(LED_E1-Pad3)
- LED_W1 pad 3: Net-(LED_E1-Pad2) -> Net-(LED_Q1-Pad2)
- LED_X1 pad 2: Net-(LED_X1-Pad2) -> Net-(LED_C1-Pad3)
- LED_X1 pad 3: Net-(LED_C1-Pad2) -> Net-(LED_X1-Pad3)
- LED_Y1 pad 2: Net-(LED_T1-Pad3) -> Net-(LED_U1-Pad3)
- LED_Y1 pad 3: Net-(LED_U1-Pad2) -> Net-(LED_T1-Pad2)
- LED_Z1 pad 2: Net-(LED_Z1-Pad2) -> Net-(LED_X1-Pad3)
- LED_Z1 pad 3: Net-(LED_X1-Pad2) -> Net-(LED_Z1-Pad3)
- LED_backspace1 pad 2: Net-(LED_backslash1-Pad3) -> Net-(LED_backspace1-Pad2)
- LED_backspace1 pad 3: Net-(LED_backspace1-Pad3) -> Net-(LED_backslash1-Pad2)
- LED_capsLock1 pad 2: Net-(LED_A1-Pad3) -> Net-(LED_capsLock1-Pad2)
- LED_capsLock1 pad 3: Net-(LED_capsLock1-Pad3) -> Net-(LED_A1-Pad2)
- LED_closeBracket1 pad 2: Net-(LED_closeBracket1-Pad2) -> Net-(LED_backslash1-Pad3)
- LED_closeBracket1 pad 3: Net-(LED_backslash1-Pad2) -> Net-(LED_closeBracket1-Pad3)
- LED_colon1 pad 2: Net-(LED_colon1-Pad2) -> Net-(LED_L1-Pad3)
- LED_colon1 pad 3: Net-(LED_L1-Pad2) -> Net-(LED_colon1-Pad3)
- LED_comma1 pad 2: Net-(LED_M1-Pad3) -> Net-(LED_comma1-Pad2)
- LED_comma1 pad 3: Net-(LED_comma1-Pad3) -> Net-(LED_M1-Pad2)
- LED_delete1 pad 2: Net-(LED_F12-Pad3) -> unconnected-(LED_delete1-Pad2)
- LED_delete1 pad 3: Net-(LED_delete1-Pad3) -> Net-(LED_F12-Pad2)
- LED_end1 pad 2: Net-(LED_end1-Pad2) -> Net-(LED_rightArrow1-Pad3)
- LED_end1 pad 3: RGBLED -> Net-(LED_end1-Pad3)
- LED_equals1 pad 2: Net-(LED_backspace1-Pad3) -> Net-(LED_equals1-Pad2)
- LED_equals1 pad 3: Net-(LED_equals1-Pad3) -> Net-(LED_backspace1-Pad2)
- LED_esc1 pad 2: Net-(LED_esc1-Pad2) -> Net-(LED_F1-Pad3)
- LED_esc1 pad 3: Net-(LED_F1-Pad2) -> Net-(LED_esc1-Pad3)
- LED_home1 pad 2: Net-(LED_delete1-Pad3) -> Net-(LED_home1-Pad2)
- LED_home1 pad 3: Net-(LED_home1-Pad3) -> RGBLED
- LED_leftArrow1 pad 2: Net-(LED_downArrow1-Pad3) -> Net-(LED_leftArrow1-Pad2)
- LED_leftArrow1 pad 3: Net-(LED_leftArrow1-Pad3) -> Net-(LED_downArrow1-Pad2)
- LED_leftShift1 pad 2: Net-(LED_leftControl1-Pad3) -> Net-(LED_Z1-Pad3)
- LED_leftShift1 pad 3: Net-(LED_Z1-Pad2) -> Net-(LED_leftControl1-Pad2)
- LED_minus1 pad 2: Net-(LED_equals1-Pad3) -> Net-(LED_0-Pad3)
- LED_minus1 pad 3: Net-(LED_0-Pad2) -> Net-(LED_equals1-Pad2)
- LED_openBracket1 pad 2: Net-(LED_P1-Pad3) -> Net-(LED_closeBracket1-Pad3)
- LED_openBracket1 pad 3: Net-(LED_closeBracket1-Pad2) -> Net-(LED_P1-Pad2)
- LED_period1 pad 2: Net-(LED_comma1-Pad3) -> Net-(LED_period1-Pad2)
- LED_period1 pad 3: Net-(LED_period1-Pad3) -> Net-(LED_comma1-Pad2)
- LED_pgDn1 pad 2: Net-(LED_pgDn1-Pad2) -> Net-(LED_end1-Pad3)
- LED_pgDn1 pad 3: Net-(LED_end1-Pad2) -> Net-(LED_pgDn1-Pad3)
- LED_pgUp1 pad 2: Net-(LED_home1-Pad3) -> Net-(LED_pgDn1-Pad3)
- LED_pgUp1 pad 3: Net-(LED_pgDn1-Pad2) -> Net-(LED_home1-Pad2)
- LED_questionMark1 pad 2: Net-(LED_period1-Pad3) -> Net-(LED_questionMark1-Pad2)
- LED_questionMark1 pad 3: Net-(LED_questionMark1-Pad3) -> Net-(LED_period1-Pad2)
- LED_quote1 pad 2: Net-(LED_enter1-Pad3) -> Net-(LED_colon1-Pad3)
- LED_quote1 pad 3: Net-(LED_colon1-Pad2) -> Net-(LED_enter1-Pad2)
- LED_rightAlt1 pad 2: Net-(LED_function1-Pad3) -> Net-(LED_rightAlt1-Pad2)
- LED_rightAlt1 pad 3: Net-(LED_rightAlt1-Pad3) -> Net-(LED_function1-Pad2)
- LED_rightArrow1 pad 2: unconnected-(LED_rightArrow1-Pad2) -> Net-(LED_downArrow1-Pad3)
- LED_rightArrow1 pad 3: Net-(LED_downArrow1-Pad2) -> Net-(LED_rightArrow1-Pad3)
- LED_rightControl1 pad 2: Net-(LED_leftArrow1-Pad3) -> Net-(LED_function1-Pad3)
- LED_rightControl1 pad 3: Net-(LED_function1-Pad2) -> Net-(LED_leftArrow1-Pad2)
- LED_rightShift1 pad 2: Net-(LED_questionMark1-Pad3) -> Net-(LED_rightShift1-Pad2)
- LED_rightShift1 pad 3: Net-(LED_rightShift1-Pad3) -> Net-(LED_questionMark1-Pad2)
- LED_space1 pad 2: Net-(LED_rightAlt1-Pad3) -> Net-(LED_leftAlt1-Pad3)
- LED_space1 pad 3: Net-(LED_leftAlt1-Pad2) -> Net-(LED_rightAlt1-Pad2)
- LED_tab1 pad 2: Net-(LED_capsLock1-Pad3) -> Net-(LED_Q1-Pad3)
- LED_tab1 pad 3: Net-(LED_Q1-Pad2) -> Net-(LED_capsLock1-Pad2)
- LED_tilda1 pad 2: Net-(LED_1-Pad3) -> Net-(LED_esc1-Pad3)
- LED_tilda1 pad 3: Net-(LED_esc1-Pad2) -> Net-(LED_1-Pad2)
- LED_upArrow1 pad 2: Net-(LED_rightShift1-Pad3) -> Net-(LED_enter1-Pad3)
- LED_upArrow1 pad 3: Net-(LED_enter1-Pad2) -> Net-(LED_rightShift1-Pad2)
- LED_windows1 pad 2: Net-(LED_leftAlt1-Pad3) -> Net-(LED_leftControl1-Pad3)
- LED_windows1 pad 3: Net-(LED_leftControl1-Pad2) -> Net-(LED_leftAlt1-Pad2)
- R4 pad 1: Net-(J1-PadA6) -> GND
- U1 pad 10: ROW4 -> COL14
- U1 pad 11: ROW5 -> ROW4
- U1 pad 12: RGBLED -> ROW5
- U1 pad 9: COL14 -> RGBLED
- U2 pad 1: GND -> unconnected-(U2-Pad1)
- U2 pad 2: Net-(J1-PadA6) -> GND
Routing:
- net Net-(LED_rightAlt1-Pad3): track 64.2 -> 0.00 mm
- net Net-(LED_rightAlt1-Pad2): track 0.00 -> 64.2 mm
- net Net-(LED_leftAlt1-Pad3): track 19.1 -> 66.6 mm
- net Net-(LED_leftAlt1-Pad2): track 66.6 -> 19.1 mm
- net Net-(LED_end1-Pad2): track 40.9 -> 0.00 mm
- net GND: track 2140.0 -> 2099.2 mm
- net Net-(LED_pgDn1-Pad2): track 40.3 -> 0.00 mm
- net Net-(LED_delete1-Pad3): track 34.3 -> 0.00 mm
- net Net-(LED_rightArrow1-Pad3): track 0.00 -> 33.0 mm
- net Net-(LED_end1-Pad3): track 0.00 -> 31.0 mm
- net Net-(LED_pgDn1-Pad3): track 0.00 -> 30.4 mm
- net Net-(LED_esc1-Pad3): track 0.00 -> 30.0 mm
- net Net-(LED_esc1-Pad2): track 30.0 -> 0.00 mm
- net Net-(LED_home1-Pad2): track 0.00 -> 28.8 mm
- net Net-(LED_rightShift1-Pad3): track 28.2 -> 0.00 mm
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
Commit message: Finished trace routing
Parts:
- moved C5 2.22 mm to (344.6, 146.5)
- moved R1 2.15 mm to (345.7, 147.6)
- moved C1 1.68 mm to (334.7, 140.3)
- moved Y1 1.36 mm to (337.4, 143.1)
- moved C2 1.30 mm to (340.1, 145.7)
Connections:
- J1 pad A6: GND -> Net-(J1-PadA6)
- J1 pad B6: GND -> Net-(J1-PadA6)
- R4 pad 1: GND -> Net-(J1-PadA6)
- U2 pad 1: unconnected-(U2-Pad1) -> GND
- U2 pad 2: GND -> Net-(J1-PadA6)
Routing:
- net GND: track 2099.2 -> 2203.2 mm, vias 0 -> 4
- net Net-(J1-PadA6): track 0.00 -> 9.61 mm
- net +5V: track 2106.5 -> 2115.1 mm, vias 7 -> 8
- net Net-(C1-Pad1): track 9.50 -> 7.42 mm
- net Net-(C2-Pad1): track 11.1 -> 9.98 mm
- net Net-(R1-Pad2): track 18.2 -> 19.0 mm
- net D+: track 65.7 -> 65.0 mm
- net D-: track 64.6 -> 63.8 mm

Commit message: silkscreen
Other:
- board text added: "Jupiter"
- board text added: "Keyboard PCB Rev 1.0 7/8/2022"
Changed lines of the file:
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@@
   (gr_line (start 366.060859 191.418837) (end 60.481213 191.458638) (layer "Edge.Cuts") (width 0.1))
   (gr_line (start 370.50005 72.097779) (end 370.558638 187.118787) (layer "Edge.Cuts") (width 0.1))
+  (gr_text "Jupiter" (at 112.1 89) (layer "B.SilkS")
+    (effects (font (size 6 6) (thickness 0.5)) (justify mirror))
+  )
+  (gr_text "Keyboard PCB Rev 1.0 7/8/2022" (at 83.8 91.4) (layer "B.SilkS")
+    (effects (font (size 1 1) (thickness 0.15)) (justify mirror))
+  )
+  (gr_text "Jupiter" (at 86.13 89.05) (layer "F.SilkS")
+    (effects (font (size 6 6) (thickness 0.5)))
+  )
+  (gr_text "Keyboard PCB Rev 1.0 7/8/2022" (at 114 91.4) (layer "F.SilkS")
+    (effects (font (size 1 1) (thickness 0.15)))
+  )
   (segment (start 343.7 79.6) (end 343.7 84.7) (width 0.25) (layer "F.Cu") (net 1))
   (segment (start 360.38 168.87) (end 360.38 168.67) (width 0.25) (layer "F.Cu") (net 1))

Commit message: Added mounting holes
Parts:
- added ?: MountingHole_2.5mm_Pad, MountingHole:MountingHole_2.5mm_Pad, F.Cu at (304.8, 97.5)
- added ?: MountingHole_2.5mm_Pad, MountingHole:MountingHole_2.5mm_Pad, F.Cu at (239.3, 74.2)
- added ?: MountingHole_2.5mm_Pad, MountingHole:MountingHole_2.5mm_Pad, F.Cu at (296.3, 149.5)
- added ?: MountingHole_2.5mm_Pad, MountingHole:MountingHole_2.5mm_Pad, F.Cu at (60.1, 187.7)
- added ?: MountingHole_2.5mm_Pad, MountingHole:MountingHole_2.5mm_Pad, F.Cu at (366.3, 71.6)
- added ?: MountingHole_2.5mm_Pad, MountingHole:MountingHole_2.5mm_Pad, F.Cu at (367.2, 187.9)
- added ?: MountingHole_2.5mm_Pad, MountingHole:MountingHole_2.5mm_Pad, F.Cu at (246.4, 110.0)
- added ?: MountingHole_2.5mm_Pad, MountingHole:MountingHole_2.5mm_Pad, F.Cu at (222.9, 148.1)
- added ?: MountingHole_2.5mm_Pad, MountingHole:MountingHole_2.5mm_Pad, F.Cu at (151.7, 92.4)
- added ?: MountingHole_2.5mm_Pad, MountingHole:MountingHole_2.5mm_Pad, F.Cu at (127.6, 148.1)
- added ?: MountingHole_2.5mm_Pad, MountingHole:MountingHole_2.5mm_Pad, F.Cu at (77.1, 75.0)
- added ?: MountingHole_2.5mm_Pad, MountingHole:MountingHole_2.5mm_Pad, F.Cu at (81.7, 114.0)
Routing:
- net GND: track 2203.2 -> 2200.2 mm
- net Net-(LED_rightArrow1-Pad3): track 33.0 -> 32.1 mm
- net +5V: track 2115.1 -> 2114.2 mm
